File: CBB-XBEE-r02.sch (EAGLE design)
At the start: 35 parts, among them IC1 TLV1117-XX, J1 HEADER_1X23, J10 HEADER_1X9, J11 HEADER_1X9, J12 HEADER_1X1, J13 HEADER_1X1, J14 HEADER_1X2, J15 HEADER_1X1, J16 HEADER_1X1, J17 HEADER_1X1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

Commit message: modified layout to include extra test points for series 3 xbees.
Parts:
- added J19, J20, J21: HEADER_1X1, logic-supply:HEADER_1X1
- C1, C2, C3: device logic-supply:C1206 -> logic-supply:C0805
- LED1, LED2: device SparkFun-LED:LED3MM -> adafruit:LEDCHIPLED_0805
- R1, R2: device logic-supply:R1206 -> logic-supply:R0805
- R3, R4: device logic-supply:R0207/10 -> logic-supply:R0805
Connections:
- net RADIO_P12 renamed CTS
- net RADIO_P16 renamed RTS
- new net DIO3: J19.1, RADIO1.DIO3
- new net ON_!SLEEP: J21.1, RADIO1.DIO9
- new net SLEEP_RQ: J20.1, RADIO1.DTR
Other:
- note added: "TLV1117‑33IDCY"
